File: schematic/KiCad/IoTeX-Devboard.sch (KiCad schematic (older format))
At the start: 93 parts, among them J1 Conn_02x05_Odd_Even, J2 USB, J3 TE 2337019-1, J4 SIM_Card_small, J5 SC_FW_UPD, J6 Conn_01x02, Q1 PMOS, Q2 PMOS, Q3 PMOS, U1 KTD2026_LED_Driver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

Commit message: IoTeX-Devboard v0.2 - Fixed STS line and Voltage Detector
IoTeX-Devboard v0.2
- Changed R21 value to 1k
- Changed R20 value to 1.5k
- Added Q4 and R25 level shifter
- STS signal shifted with Q4 instead U11
- Added C35 bypass capacitor
Parts:
- added C35: 0.1u, Capacitor_SMD:C_0402_1005Metric, symbol Device:C_Small
- added PB3: K2-1107UT-A45W-06, STETEL_Devices:SW_SPST_PTS815, symbol Switch:SW_Push
- added Q4: NMOS, symbol Device:Q_NMOS_GSD
- added R24: 1k, Resistor_SMD:R_0402_1005Metric, symbol Device:R_Small_US
- added R25: 100k, Resistor_SMD:R_0402_1005Metric, symbol Device:R_Small_US
- R20: value 150k -> 1.5k
- R21: value 100k -> 1k
Connections:
- net GND: now also C35.1, PB3.2, Q4.2 (S)
- net LV_STS: now also Q4.1 (G); no longer U11.5 (A4)
- net SC_PWK: now also R24.2; no longer J1.3 (Pin_3)
- net SC_STS: now also Q4.3 (D), R25.1; no longer U11.10 (B4)
- net at U7.12 (VIN), U7.15 (VOUT): now also C35.2
- new net BOOT: J1.3 (Pin_3), PB3.1, R24.1
- no-connect marks 43 -> 45
Other:
- moved on the sheet: C24, C30, D2, D3, J5, R18, U11
